File: Xadow MultiSerial.sch (EAGLE design)
At the start: 19 parts, among them J1 12p 0.5mm bottom contact, J2 12p 0.5mm bottom contact, J3 12p 0.5mm bottom contact, J4 12p 0.5mm bottom contact, U1 SC16IS752, X1 CTS_32X25_SMD

Commit message: Added level shifter MOSFETs
Parts:
- added Q1, Q2, Q3, Q4, Q5, Q6: MOSFET-N-044020001, OPL:MOSFET-N-044020001
- added R10, R11, R12, R13, R14, R15, R16, R17, R18, R7, R8, R9: 10K, OPL:R-0603
Connections:
- new net N$11: Q1.S, R7.1
- new net N$12: Q2.S, R9.1
- new net N$13: Q3.S, R11.1
- new net N$14: Q4.S, R13.1
- new net N$15: Q5.S, R15.1
- new net N$16: Q6.S, R17.1
- new net N$17: R10.2, R12.2, R14.2, R16.2, R18.2, R8.2
- new net N$18: Q1.D, R8.1
- new net N$19: Q2.D, R10.1
- new net N$20: Q3.D, R12.1
- new net N$21: Q4.D, R14.1
- new net N$22: Q5.D, R16.1
- new net N$23: Q6.D, R18.1
- new net N$4: Q1.G, Q2.G, Q3.G, Q4.G, Q5.G, Q6.G, R11.2, R13.2, R15.2, R17.2, R7.2, R9.2
Other:
- moved on the sheet: D1, D2, D3, D4, R3, R4, R5, R6

Commit message: Arranged level shifter mosfets
Parts:
- added PAD1, PAD2, PAD3, PAD4, PAD5, PAD6, PAD7, PAD8: WIREPADSMD1,27-254, wirepad:WIREPADSMD1,27-254
Connections:
- net GND: now also PAD8.P
- net N$18: now also PAD2.P
- net N$19: now also PAD1.P
- net N$20: now also PAD3.P
- net N$21: now also PAD4.P
- net N$22: now also PAD5.P
- net N$23: now also PAD6.P
- net N$4: now also PAD7.P
Changed lines of the file:
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@@
 <part name="R17" library="OPL" deviceset="R*" device="-0603" value="10K"/>
 <part name="R18" library="OPL" deviceset="R*" device="-0603" value="10K"/>
+<part name="PAD1" library="wirepad" deviceset="WIREPAD" device="SMD1,27-254"/>
+<part name="PAD2" library="wirepad" deviceset="WIREPAD" device="SMD1,27-254"/>
+<part name="PAD3" library="wirepad" deviceset="WIREPAD" device="SMD1,27-254"/>
+<part name="PAD4" library="wirepad" deviceset="WIREPAD" device="SMD1,27-254"/>
+<part name="PAD5" library="wirepad" deviceset="WIREPAD" device="SMD1,27-254"/>
+<part name="PAD6" library="wirepad" deviceset="WIREPAD" device="SMD1,27-254"/>
+<part name="PAD7" library="wirepad" deviceset="WIREPAD" device="SMD1,27-254"/>
+<part name="PAD8" library="wirepad" deviceset="WIREPAD" device="SMD1,27-254"/>
+<part name="GND3" library="supply1" deviceset="GND" device=""/>
 </parts>
 <sheets>
@@
 <instance part="R17" gate="R" x="172.72" y="91.44" rot="R90"/>
 <instance part="R18" gate="R" x="182.88" y="91.44" rot="R90"/>
+<instance part="PAD1" gate="G$1" x="132.08" y="76.2" smashed="yes" rot="R90">
+<attribute name="NAME" x="130.2258" y="75.057" size="1.778" layer="95" rot="R90"/>
+</instance>
+<instance part="PAD2" gate="G$1" x="119.38" y="76.2" smashed="yes" rot="R90">
+<attribute name="NAME" x="117.5258" y="75.057" size="1.778" layer="95" rot="R90"/>
+</instance>
+<instance part="PAD3" gate="G$1" x="144.78" y="76.2" smashed="yes" rot="R90">
+<attribute name="NAME" x="142.9258" y="75.057" size="1.778" layer="95" rot="R90"/>
+</instance>
+<instance part="PAD4" gate="G$1" x="157.48" y="76.2" smashed="yes" rot="R90">
+<attribute name="NAME" x="155.6258" y="75.057" size="1.778" layer="95" rot="R90"/>
+</instance>
+<instance part="PAD5" gate="G$1" x="170.18" y="76.2" smashed="yes" rot="R90">
+<attribute name="NAME" x="168.3258" y="75.057" size="1.778" layer="95" rot="R90"/>
+</instance>
+<instance part="PAD6" gate="G$1" x="182.88" y="76.2" smashed="yes" rot="R90">
+<attribute name="NAME" x="181.0258" y="75.057" size="1.778" layer="95" rot="R90"/>
+</instance>
+<instance part="PAD7" gate="G$1" x="99.06" y="101.6" smashed="yes">
+<attribute name="NAME" x="97.917" y="103.4542" size="1.778" layer="95"/>
+</instance>
+<instance part="PAD8" gate="G$1" x="88.9" y="88.9" smashed="yes">
+<attribute name="NAME" x="87.757" y="90.7542" size="1.778" layer="95"/>
+</instance>
+<instance part="GND3" gate="1" x="98.806" y="88.9" rot="R90"/>
 </instances>
 <busses>
@@
 <pinref part="GND2" gate="1" pin="GND"/>
 <junction x="159.258" y="115.316"/>
+</segment>
+<segment>
+<pinref part="PAD8" gate="G$1" pin="P"/>
+<pinref part="GND3" gate="1" pin="GND"/>
+<wire x1="96.266" y1="88.9" x2="91.44" y2="88.9" width="0.1524" layer="91"/>
 </segment>
 </net>
@@
 <pinref part="R15" gate="R" pin="2"/>
 <pinref part="R17" gate="R" pin="2"/>
+<pinref part="PAD7" gate="G$1" pin="P"/>
 </segment>
 </net>
@@
 <pinref part="R7" gate="R" pin="1"/>
 <wire x1="109.22" y1="87.63" x2="109.22" y2="86.36" width="0.1524" layer="91"/>
+<wire x1="109.22" y1="86.36" x2="109.22" y2="78.74" width="0.1524" layer="91"/>
+<junction x="109.22" y="86.36"/>
 </segment>
 </net>
@@
 <pinref part="R9" gate="R" pin="1"/>
 <wire x1="121.92" y1="87.63" x2="121.92" y2="86.36" width="0.1524" layer="91"/>
+<wire x1="121.92" y1="86.36" x2="121.92" y2="78.74" width="0.1524" layer="91"/>
+<junction x="121.92" y="86.36"/>
 </segment>
 </net>
@@
 <pinref part="R11" gate="R" pin="1"/>
 <wire x1="134.62" y1="87.63" x2="134.62" y2="86.36" width="0.1524" layer="91"/>
+<wire x1="134.62" y1="86.36" x2="134.62" y2="78.74" width="0.1524" layer="91"/>
+<junction x="134.62" y="86.36"/>
 </segment>
 </net>
@@
 <pinref part="R13" gate="R" pin="1"/>
 <wire x1="147.32" y1="87.63" x2="147.32" y2="86.36" width="0.1524" layer="91"/>
+<wire x1="147.32" y1="86.36" x2="147.32" y2="78.74" width="0.1524" layer="91"/>
+<junction x="147.32" y="86.36"/>
 </segment>
 </net>
@@
 <pinref part="R15" gate="R" pin="1"/>
 <wire x1="160.02" y1="87.63" x2="160.02" y2="86.36" width="0.1524" layer="91"/>
+<wire x1="160.02" y1="86.36" x2="160.02" y2="78.74" width="0.1524" layer="91"/>
+<junction x="160.02" y="86.36"/>
 </segment>
 </net>
@@
 <pinref part="R17" gate="R" pin="1"/>
 <wire x1="172.72" y1="87.63" x2="172.72" y2="86.36" width="0.1524" layer="91"/>
+<wire x1="172.72" y1="86.36" x2="172.72" y2="78.74" width="0.1524" layer="91"/>
+<junction x="172.72" y="86.36"/>
 </segment>
 </net>
@@
 <wire x1="119.38" y1="86.36" x2="119.38" y2="87.63" width="0.1524" layer="91"/>
 <pinref part="R8" gate="R" pin="1"/>
+<wire x1="119.38" y1="86.36" x2="119.38" y2="78.74" width="0.1524" layer="91"/>
+<junction x="119.38" y="86.36"/>
+<pinref part="PAD2" gate="G$1" pin="P"/>
 </segment>
 </net>
@@
 <wire x1="132.08" y1="86.36" x2="132.08" y2="87.63" width="0.1524" layer="91"/>
 <pinref part="R10" gate="R" pin="1"/>
+<wire x1="132.08" y1="86.36" x2="132.08" y2="78.74" width="0.1524" layer="91"/>
+<junction x="132.08" y="86.36"/>
+<pinref part="PAD1" gate="G$1" pin="P"/>
 </segment>
 </net>
@@
 <wire x1="144.78" y1="86.36" x2="144.78" y2="87.63" width="0.1524" layer="91"/>
 <pinref part="R12" gate="R" pin="1"/>
+<wire x1="144.78" y1="86.36" x2="144.78" y2="78.74" width="0.1524" layer="91"/>
+<junction x="144.78" y="86.36"/>
+<pinref part="PAD3" gate="G$1" pin="P"/>
 </segment>
 </net>
@@
 <wire x1="157.48" y1="86.36" x2="157.48" y2="87.63" width="0.1524" layer="91"/>
 <pinref part="R14" gate="R" pin="1"/>
+<wire x1="157.48" y1="86.36" x2="157.48" y2="78.74" width="0.1524" layer="91"/>
+<junction x="157.48" y="86.36"/>
+<pinref part="PAD4" gate="G$1" pin="P"/>
 </segment>
 </net>
@@
 <wire x1="170.18" y1="86.36" x2="170.18" y2="87.63" width="0.1524" layer="91"/>
 <pinref part="R16" gate="R" pin="1"/>
+<wire x1="170.18" y1="86.36" x2="170.18" y2="78.74" width="0.1524" layer="91"/>
+<junction x="170.18" y="86.36"/>
+<pinref part="PAD5" gate="G$1" pin="P"/>
 </segment>
 </net>
@@
 <wire x1="182.88" y1="86.36" x2="182.88" y2="87.63" width="0.1524" layer="91"/>
 <pinref part="R18" gate="R" pin="1"/>
-</segment>
-</net>
+<wire x1="182.88" y1="86.36" x2="182.88" y2="78.74" width="0.1524" layer="91"/>
+<junction x="182.88" y="86.36"/>
+<pinref part="PAD6" gate="G$1" pin="P"/>
+</segment>
+</net>

Commit message: Added through hole pads and adjusted labels
Parts:
- removed PAD1, PAD2, PAD3, PAD4, PAD5, PAD6, PAD7, PAD8: WIREPADSMD1,27-254, wirepad:WIREPADSMD1,27-254
- added 5V, GND, RXA_5, RXB_5, RXI_5, TXA_5, TXB_5, TXO_5: WIREPAD1,6/0,8, wirepad:WIREPAD1,6/0,8
Connections:
- removed net N$11: Q1.S, R7.1
- removed net N$12: Q2.S, R9.1
- removed net N$13: Q3.S, R11.1
- removed net N$14: Q4.S, R13.1
- removed net N$15: Q5.S, R15.1
- removed net N$16: Q6.S, R17.1
- removed net N$4: PAD7.P, Q1.G, Q2.G, Q3.G, Q4.G, Q5.G, Q6.G, R11.2, R13.2, R15.2, R17.2, R7.2, R9.2
- net 3V3: now also Q1.G, Q2.G, Q3.G, Q4.G, Q5.G, Q6.G, R11.2, R13.2, R15.2, R17.2, R7.2, R9.2
- net GND: now also GND.P; no longer PAD8.P
- net N$17: now also 5V.P
- net N$18: now also TXB_5.P; no longer PAD2.P
- net N$19: now also RXB_5.P; no longer PAD1.P
- net N$20: now also TXA_5.P; no longer PAD3.P
- net N$21: now also RXA_5.P; no longer PAD4.P
- net N$22: now also TXO_5.P; no longer PAD5.P
- net N$23: now also RXI_5.P; no longer PAD6.P
- net PD2/RXI/D0: now also Q6.S, R17.1; no longer J1.2, J4.2
- net PD3/TXO/D1: now also Q5.S, R15.1; no longer J1.1, J4.1
- net RXA: now also J4.2, Q4.S, R13.1
- net RXB: now also J1.2, Q2.S, R9.1
- net TXA: now also J4.1, Q3.S, R11.1
- net TXB: now also J1.1, Q1.S, R7.1

Commit message: Fixed errors and relayed out, last attempt with MOSFET level shifter, need to try TXS shifter
Connections:
- net N$3: no longer R2.2
- net N$5: now also R2.2
- net PB1/D15/SCK: now also J4.1; no longer J4.12
- net PB2/D16/MOSI: now also J4.2; no longer J4.11
- net PB3/D14/MISO: now also J4.3; no longer J4.10
- net PD0/SCL/D3: now also J4.9; no longer J4.4
- net PD1/SDA/D2: now also J4.10; no longer J4.3
- net PF0/A5: now also J4.4; no longer J4.9
- net RXA: now also J4.11; no longer J4.2
- net TXA: now also J4.12; no longer J4.1
Other:
- moved on the sheet: J4, S1

Commit message: Added TXS based level translation
Parts:
- removed Q1, Q2, Q3, Q4, Q5, Q6: MOSFET-N-044020001, OPL:MOSFET-N-044020001
- removed R10, R11, R12, R13, R14, R15, R16, R17, R18, R7, R8, R9: 10K, OPL:R-0603
- removed RXA_5, RXB_5, RXI_5, TXA_5, TXB_5, TXO_5: WIREPAD1,6/0,8, wirepad:WIREPAD1,6/0,8
- added RXA, RXB, RXI, TXA, TXB, TXO: (no value), wirepad:1,6/0,8
- added U2: TXB0106PWR, Texas Instruments_By_element14_Batch_1:TXB0106PWR
- 5V, GND: value WIREPAD1,6/0,8 -> (none); device wirepad:WIREPAD1,6/0,8 -> wirepad:1,6/0,8
Connections:
- removed net N$17: 5V.P, R10.2, R12.2, R14.2, R16.2, R18.2, R8.2
- new net N$4: 5V.P, U2.VCCB
- net 3V3: now also U2.OE, U2.VCCA; no longer Q1.G, Q2.G, Q3.G, Q4.G, Q5.G, Q6.G, R11.2, R13.2, R15.2, R17.2, R7.2, R9.2
- net GND: now also U2.GND
- net N$18: now also RXI.P, U2.B1; no longer Q1.D, R8.1, TXB_5.P
- net N$19: now also TXO.P, U2.B2; no longer Q2.D, R10.1, RXB_5.P
- net N$20: now also RXA.P, U2.B3; no longer Q3.D, R12.1, TXA_5.P
- net N$21: now also TXA.P, U2.B4; no longer Q4.D, R14.1, RXA_5.P
- net N$22: now also RXB.P, U2.B5; no longer Q5.D, R16.1, TXO_5.P
- net N$23: now also TXB.P, U2.B6; no longer Q6.D, R18.1, RXI_5.P
- net PB1/D15/SCK: no longer J1.12, J4.1
- net PB2/D16/MOSI: no longer J1.11, J4.2
- net PB3/D14/MISO: no longer J1.10, J4.3
- net PD0/SCL/D3: no longer J1.4, J4.9
- net PD1/SDA/D2: no longer J1.3, J4.10
- net PD2/RXI/D0: now also U2.A1; no longer Q6.S, R17.1
- net PD3/TXO/D1: now also U2.A2; no longer Q5.S, R15.1
- net PF0/A5: no longer J1.9, J4.4
- net RXA: now also U2.A3; no longer Q4.S, R13.1
- net RXB: now also U2.A5; no longer Q2.S, R9.1
- net TXA: now also U2.A4; no longer Q3.S, R11.1
- net TXB: now also U2.A6; no longer Q1.S, R7.1

Commit message: Changed author
Other:
- note added: "Tisham Dhar"
- note added: "v1.0"
- note removed: "Albert Miao"
- note removed: "v0.1a"
Changed lines of the file:
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@@
 <sheet>
 <plain>
-<text x="191.77" y="11.43" size="1.778" layer="94" ratio="10">Albert Miao</text>
-<text x="224.79" y="5.08" size="1.778" layer="94" ratio="10">v0.1a</text>
+<text x="191.77" y="11.43" size="1.778" layer="94" ratio="10">Tisham Dhar</text>
+<text x="224.79" y="5.08" size="1.778" layer="94" ratio="10">v1.0</text>
 </plain>
 <instances>

Commit message: Changed to 5x3 crystal
Parts:
- removed X1: CTS_32X25_SMD, crystal-cts:CTS_32X25_SMD
- added Y1: (no value), SparkFun-FreqCtrl:CRYSTAL5X3
Connections:
- net GND: no longer X1.GND
- net N$1: now also Y1.1; no longer X1.X1
- net N$2: now also Y1.2; no longer X1.X2
Other:
- note added: "Albert Miao"
- note added: "v0.1a"
- note removed: "Tisham Dhar"
- note removed: "v1.0"
Changed lines of the file:
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@@
 <part name="J3" library="template" deviceset="FPC052002-12LT" device="" value="12p 0.5mm bottom contact"/>
 <part name="U$1" library="moudle" deviceset="SEEEDSTUDIO_SCH_FRAME" device=""/>
-<part name="X1" library="crystal-cts" deviceset="CTS_32X25_SMD" device=""/>
 <part name="U1" library="nxpsemi" deviceset="SC16IS752" device=""/>
 <part name="J1" library="template" deviceset="FPC052002-12LT" device="" value="12p 0.5mm bottom contact"/>
@@
 <part name="TXB" library="wirepad" deviceset="1,6/0,8" device=""/>
 <part name="GND" library="wirepad" deviceset="1,6/0,8" device=""/>
+<part name="Y1" library="SparkFun-FreqCtrl" deviceset="CRYSTAL" device="5X3"/>
 </parts>
 <sheets>
 <sheet>
 <plain>
-<text x="191.77" y="11.43" size="1.778" layer="94" ratio="10">Tisham Dhar</text>
-<text x="224.79" y="5.08" size="1.778" layer="94" ratio="10">v1.0</text>
+<text x="191.77" y="11.43" size="1.778" layer="94" ratio="10">Albert Miao</text>
+<text x="224.79" y="5.08" size="1.778" layer="94" ratio="10">v0.1a</text>
 </plain>
 <instances>
@@
 </instance>
 <instance part="U$1" gate="G$1" x="0" y="0"/>
-<instance part="X1" gate="G$2" x="173.482" y="141.478" smashed="yes" rot="R270"/>
 <instance part="U1" gate="G$1" x="214.122" y="135.128"/>
 <instance part="J1" gate="G$1" x="46.482" y="85.598" smashed="yes" rot="R180">
@@
 <instance part="TXB" gate="P" x="172.72" y="66.04" rot="R180"/>
 <instance part="GND" gate="P" x="91.44" y="55.88"/>
+<instance part="Y1" gate="G$1" x="173.482" y="141.224" rot="R270"/>
 </instances>
 <busses>
@@
 </segment>
 <segment>
-<pinref part="X1" gate="G$2" pin="GND"/>
-<wire x1="165.862" y1="141.478" x2="162.052" y2="141.478" width="0.1524" layer="91"/>
 <pinref part="C1" gate="C" pin="1"/>
 <wire x1="162.052" y1="141.478" x2="160.782" y2="141.478" width="0.1524" layer="91"/>
@@
 <wire x1="183.896" y1="140.208" x2="183.896" y2="150.876" width="0.1524" layer="91"/>
 <wire x1="183.896" y1="150.876" x2="173.482" y2="150.876" width="0.1524" layer="91"/>
-<wire x1="173.482" y1="150.876" x2="173.482" y2="149.098" width="0.1524" layer="91"/>
-<pinref part="X1" gate="G$2" pin="X1"/>
+<wire x1="173.482" y1="150.876" x2="173.482" y2="143.764" width="0.1524" layer="91"/>
 <pinref part="U1" gate="G$1" pin="XTAL1"/>
 <pinref part="C1" gate="C" pin="2"/>
@@
 <wire x1="171.45" y1="150.876" x2="171.45" y2="147.32" width="0.1524" layer="91"/>
 <junction x="173.482" y="150.876"/>
+<pinref part="Y1" gate="G$1" pin="1"/>
 </segment>
 </net>
@@
 <wire x1="183.896" y1="137.668" x2="183.896" y2="131.318" width="0.1524" layer="91"/>
 <wire x1="183.896" y1="131.318" x2="173.482" y2="131.318" width="0.1524" layer="91"/>
-<pinref part="X1" gate="G$2" pin="X2"/>
-<wire x1="173.482" y1="133.858" x2="173.482" y2="131.318" width="0.1524" layer="91"/>
 <pinref part="U1" gate="G$1" pin="XTAL2"/>
 <pinref part="C2" gate="C" pin="2"/>
+<wire x1="173.482" y1="138.684" x2="173.482" y2="131.318" width="0.1524" layer="91"/>
 <wire x1="173.482" y1="131.318" x2="171.45" y2="131.318" width="0.1524" layer="91"/>
 <wire x1="171.45" y1="131.318" x2="171.45" y2="137.16" width="0.1524" layer="91"/>
 <junction x="173.482" y="131.318"/>
-</segment>
-</net>
+<pinref part="Y1" gate="G$1" pin="2"/>
+</segment>
+</net>

Commit message: Changed caps to match crystal load
Parts:
- C1: value 22pF -> 15pF
- C2: value 33pF -> 22pF
Changed lines of the file:
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@@
 <part name="U1" library="nxpsemi" deviceset="SC16IS752" device=""/>
 <part name="J1" library="template" deviceset="FPC052002-12LT" device="" value="12p 0.5mm bottom contact"/>
-<part name="C1" library="OPL" deviceset="CAP" device="-0603" value="22pF"/>
-<part name="C2" library="OPL" deviceset="CAP" device="-0603" value="33pF"/>
+<part name="C1" library="OPL" deviceset="CAP" device="-0603" value="15pF"/>
+<part name="C2" library="OPL" deviceset="CAP" device="-0603" value="22pF"/>
 <part name="GND1" library="supply1" deviceset="GND" device=""/>
 <part name="S1" library="switch-copal" deviceset="CHS-02" device="A"/>
