File: Xadow MultiSerial.sch (EAGLE design)
At the start: 28 parts, among them J1 12p 0.5mm bottom contact, J2 12p 0.5mm bottom contact, J3 12p 0.5mm bottom contact, J4 12p 0.5mm bottom contact, U1 SC16IS752, U2 TXB0106PWR

Commit message: Added mini usb and mosfet based level shifter
Parts:
- removed RXA, RXB, RXI, TXA, TXB, TXO: (no value), wirepad:1,6/0,8
- removed Y1: (no value), SparkFun-FreqCtrl:CRYSTAL5X3
- added R7: 10K, Discrete:R-4R-1206
- added RXB_5, TXB_5: (no value), wirepad:1,6/0,8
- added X1: CTS_32X25_SMD, cts_crystal:CTS_32X25_SMD
- J1: value 12p 0.5mm bottom contact -> MINI-USB-5P-3400020P1; device template:FPC052002-12LT -> OPL Eagle Library:MINI-USB-5P-3400020P1
- U2: value TXB0106PWR -> BSS138PS; device Texas Instruments_By_element14_Batch_1:TXB0106PWR -> NXP_By_element14_Batch_1:BSS138PS
Connections:
- removed net N$18: RXI.P, U2.B1
- removed net N$19: TXO.P, U2.B2
- removed net N$20: RXA.P, U2.B3
- removed net N$21: TXA.P, U2.B4
- removed net N$22: RXB.P, U2.B5
- removed net N$23: TXB.P, U2.B6
- removed net N$4: 5V.P, U2.VCCB
- new net 5V: 5V.P, J1.VCC, R7A.1, R7B.1
- new net GPIO0: J1.DM, U1.GPIO0/DSRB
- new net GPIO1: J1.ID, U1.GPIO1/DTRB
- new net RXB_5: R7A.2, RXB_5.P, U2.D1
- new net TXB_5: J1.DP, R7B.2, TXB_5.P, U2.D2
- net 3V3: now also R7C.2, R7D.2, U2.G1, U2.G2; no longer J1.5, J1.8, U2.OE, U2.VCCA
- net GND: now also J1.GND@1, J1.GND@2, J1.GND@3, J1.GND@4, J1.GND@5, X1.GND; no longer J1.6, J1.7, J1.P1, J1.P2, U2.GND
- net N$1: now also X1.X1; no longer Y1.1
- net N$2: now also X1.X2; no longer Y1.2
- net PD2/RXI/D0: no longer U2.A1
- net PD3/TXO/D1: no longer U2.A2
- net RXA: no longer U2.A3
- net RXB: now also R7C.1, U2.S1; no longer J1.2, U2.A5
- net TXA: no longer U2.A4
- net TXB: now also R7D.1, U2.S2; no longer J1.1, U2.A6
Other:
- note added: "Tisham Dhar"
- note removed: "Albert Miao"
- moved on the sheet: GND

Commit message: Converted board to SPI
Parts:
- removed R1: 10k, OPL:R-0603
- removed R2: 10K, OPL:R-0603
- removed S1: CHS-02A, switch-copal:CHS-02A
Connections:
- removed net N$3: R1.2, S1.3, U1.A1/SI
- removed net N$5: R2.2, S1.4, U1.A0/CS
- net 3V3: no longer S1.1, S1.2, U1.I2C/SPI
- net GND: now also U1.I2C/SPI, U1.SDA/VSS; no longer R1.1, R2.1
- net PB1/D15/SCK: now also U1.SCL/SCLK
- net PB2/D16/MOSI: now also U1.A1/SI
- net PB3/D14/MISO: now also U1.NC/SO
- net PD0/SCL/D3: no longer U1.SCL/SCLK
- net PD1/SDA/D2: no longer U1.SDA/VSS
- net PF0/A5: now also U1.A0/CS

Commit message: Added a 3V3 LDO to grab power
Parts:
- added C3, C4: 10uF, adafruit:C-USC0805K
- added IC2: LP298XS, adafruit:LP298XS
Connections:
- removed net 3V3: D1.+, D2.+, D3.+, D4.+, J2.5, J2.8, J3.5, J3.8, J4.5, J4.8, R7C.2, R7D.2, U1./RESET, U1.VDD, U2.G1, U2.G2
- removed net 5V: 5V.P, J1.VCC, R7A.1, R7B.1
- new net +3V3: C3.1, C4.1, D1.+, D2.+, D3.+, D4.+, IC2.VOUT, J2.5, J2.8, J3.5, J3.8, J4.5, J4.8, R7C.2, R7D.2, U1./RESET, U1.VDD, U2.G1, U2.G2
- new net +5V: 5V.P, IC2.EN, IC2.VIN, J1.VCC, R7A.1, R7B.1
- net GND: now also C3.2, C4.2, IC2.GND
Changed lines of the file:
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@@
 <part name="U2" library="NXP_By_element14_Batch_1" deviceset="BSS138PS" device=""/>
 <part name="R7" library="Discrete" deviceset="R-4R*" device="-1206" value="10K"/>
+<part name="GND3" library="supply1" deviceset="GND" device=""/>
+<part name="C3" library="adafruit" deviceset="C-US" device="C0805K" value="10uF"/>
+<part name="+3V4" library="supply1" deviceset="+3V3" device=""/>
+<part name="C4" library="adafruit" deviceset="C-US" device="C0805K" value="10uF"/>
+<part name="+3V5" library="supply1" deviceset="+3V3" device=""/>
+<part name="GND4" library="supply1" deviceset="GND" device=""/>
+<part name="IC2" library="adafruit" deviceset="LP298X" device="S"/>
+<part name="P+1" library="supply1" deviceset="+5V" device=""/>
+<part name="+3V6" library="supply1" deviceset="+3V3" device=""/>
+<part name="GND7" library="supply1" deviceset="GND" device=""/>
 </parts>
 <sheets>
@@
 <instance part="R7" gate="C" x="172.72" y="88.9"/>
 <instance part="R7" gate="D" x="172.72" y="86.36"/>
+<instance part="GND3" gate="1" x="109.22" y="25.4"/>
+<instance part="C3" gate="G$1" x="109.22" y="33.02"/>
+<instance part="+3V4" gate="G$1" x="109.22" y="38.1"/>
+<instance part="C4" gate="G$1" x="119.38" y="33.02"/>
+<instance part="+3V5" gate="G$1" x="119.38" y="38.1"/>
+<instance part="GND4" gate="1" x="119.38" y="25.4"/>
+<instance part="IC2" gate="G$1" x="58.42" y="35.56" rot="R270"/>
+<instance part="P+1" gate="1" x="35.56" y="53.34"/>
+<instance part="+3V6" gate="G$1" x="71.12" y="53.34"/>
+<instance part="GND7" gate="1" x="40.64" y="35.56" rot="R270"/>
 </instances>
 <busses>
@@
 <pinref part="GND2" gate="1" pin="GND"/>
 </segment>
-</net>
-<net name="3V3" class="2">
+<segment>
+<pinref part="C3" gate="G$1" pin="2"/>
+<pinref part="GND3" gate="1" pin="GND"/>
+</segment>
+<segment>
+<pinref part="C4" gate="G$1" pin="2"/>
+<pinref part="GND4" gate="1" pin="GND"/>
+</segment>
+<segment>
+<pinref part="IC2" gate="G$1" pin="GND"/>
+<pinref part="GND7" gate="1" pin="GND"/>
+</segment>
+</net>
+<net name="+3V3" class="2">
 <segment>
 <wire x1="8.89" y1="147.066" x2="27.94" y2="147.066" width="0.1524" layer="91"/>
@@
 <label x="175.26" y="88.9" size="1.778" layer="95" rot="R90" xref="yes"/>
 </segment>
+<segment>
+<pinref part="C3" gate="G$1" pin="1"/>
+<pinref part="+3V4" gate="G$1" pin="+3V3"/>
+</segment>
+<segment>
+<pinref part="C4" gate="G$1" pin="1"/>
+<pinref part="+3V5" gate="G$1" pin="+3V3"/>
+</segment>
+<segment>
+<wire x1="71.12" y1="50.8" x2="71.12" y2="40.64" width="0.1524" layer="91"/>
+<wire x1="71.12" y1="40.64" x2="68.58" y2="40.64" width="0.1524" layer="91"/>
+<pinref part="+3V6" gate="G$1" pin="+3V3"/>
+<pinref part="IC2" gate="G$1" pin="VOUT"/>
+</segment>
 </net>
 <net name="PB1/D15/SCK" class="0">
@@
 </segment>
 </net>
-<net name="5V" class="0">
+<net name="+5V" class="0">
 <segment>
 <pinref part="J1" gate="USB" pin="VCC"/>
@@
 <label x="106.68" y="83.82" size="1.778" layer="95" xref="yes"/>
 </segment>
-</net>
+<segment>
+<wire x1="35.56" y1="50.8" x2="35.56" y2="40.64" width="0.1524" layer="91"/>
+<wire x1="35.56" y1="40.64" x2="43.18" y2="40.64" width="0.1524" layer="91"/>
+<wire x1="35.56" y1="40.64" x2="35.56" y2="30.48" width="0.1524" layer="91"/>
+<wire x1="35.56" y1="30.48" x2="43.18" y2="30.48" width="0.1524" layer="91"/>
+<junction x="35.56" y="40.64"/>
+<pinref part="IC2" gate="G$1" pin="VIN"/>
+<pinref part="P+1" gate="1" pin="+5V"/>
+<pinref part="IC2" gate="G$1" pin="EN"/>
+</segment>
+</net>
