File: Xadow MultiSerial.brd (EAGLE design)
At the start: 25.4 x 20.3 mm, 19 parts, among them J1 12p 0.5mm bottom contact, J2 12p 0.5mm bottom contact, J3 12p 0.5mm bottom contact, J4 12p 0.5mm bottom contact, U1 SC16IS752, X1 CTS_32X25_SMD

Commit message: Added level shifter MOSFETs
Parts:
- added Q1, Q2, Q3, Q4, Q5, Q6: MOSFET-N-044020001, OPL:SOT23
- added R10, R11, R12, R13, R14, R15, R16, R17, R18, R7, R8, R9: 10K, OPL:R0603
Connections:
- new net N$11: Q1.2, R7.1
- new net N$12: Q2.2, R9.1
- new net N$13: Q3.2, R11.1
- new net N$14: Q4.2, R13.1
- new net N$15: Q5.2, R15.1
- new net N$16: Q6.2, R17.1
- new net N$17: R10.2, R12.2, R14.2, R16.2, R18.2, R8.2
- new net N$18: Q1.3, R8.1
- new net N$19: Q2.3, R10.1
- new net N$20: Q3.3, R12.1
- new net N$21: Q4.3, R14.1
- new net N$22: Q5.3, R16.1
- new net N$23: Q6.3, R18.1
- new net N$4: Q1.1, Q2.1, Q3.1, Q4.1, Q5.1, Q6.1, R11.2, R13.2, R15.2, R17.2, R7.2, R9.2
Other:
- board text added: "Xadow Multiserial"
- board text added: "v1.0 14/09/2014"
- board text removed: "Breakout"
- board text removed: "Xadow"
- board text removed: "v1.0 03/19/2013"

Commit message: Arranged level shifter mosfets
Parts:
- added PAD1, PAD2, PAD3, PAD4, PAD5, PAD6, PAD7, PAD8: WIREPADSMD1,27-254, wirepad:SMD1,27-2,54
- moved R14 19.8 mm to (22.9, 17.9)
- moved R13 19.3 mm to (22.9, 15.0)
- moved Q1 16.5 mm to (4.32, 16.4)
- moved Q2 16.3 mm to (4.32, 13.0)
- moved Q3 16.3 mm to (4.32, 9.40)
- moved R16 9.57 mm to (22.9, 7.75), turned to 180 degrees
- moved R18 7.04 mm to (20.6, 13.1)
- moved R10 7.03 mm to (6.86, 7.75)
- moved R17 6.91 mm to (20.6, 9.40)
- moved R15 3.78 mm to (22.9, 11.4), turned to 180 degrees
- moved R12 3.64 mm to (9.40, 13.1), turned to 90 degrees
- moved R11 2.61 mm to (9.40, 9.53), turned to 90 degrees
- moved R7 2.53 mm to (6.86, 14.7)
- moved Q6 1.78 mm to (25.3, 9.40)
- moved R8 1.76 mm to (6.86, 17.9)
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Connections:
- net GND: now also PAD8.1
- net N$18: now also PAD2.1
- net N$19: now also PAD1.1
- net N$20: now also PAD3.1
- net N$21: now also PAD4.1
- net N$22: now also PAD5.1
- net N$23: now also PAD6.1
- net N$4: now also PAD7.1

Commit message: Added through hole pads and adjusted labels
Parts:
- removed PAD1, PAD2, PAD3, PAD4, PAD5, PAD6, PAD7, PAD8: WIREPADSMD1,27-254, wirepad:SMD1,27-2,54
- added 5V, GND, RXA_5, RXB_5, RXI_5, TXA_5, TXB_5, TXO_5: WIREPAD1,6/0,8, wirepad:1,6/0,8
Connections:
- removed net N$11: Q1.2, R7.1
- removed net N$12: Q2.2, R9.1
- removed net N$13: Q3.2, R11.1
- removed net N$14: Q4.2, R13.1
- removed net N$15: Q5.2, R15.1
- removed net N$16: Q6.2, R17.1
- removed net N$4: PAD7.1, Q1.1, Q2.1, Q3.1, Q4.1, Q5.1, Q6.1, R11.2, R13.2, R15.2, R17.2, R7.2, R9.2
- net 3V3: now also Q1.1, Q2.1, Q3.1, Q4.1, Q5.1, Q6.1, R11.2, R13.2, R15.2, R17.2, R7.2, R9.2
- net GND: now also GND.1; no longer PAD8.1
- net N$17: now also 5V.1
- net N$18: now also TXB_5.1; no longer PAD2.1
- net N$19: now also RXB_5.1; no longer PAD1.1
- net N$20: now also TXA_5.1; no longer PAD3.1
- net N$21: now also RXA_5.1; no longer PAD4.1
- net N$22: now also TXO_5.1; no longer PAD5.1
- net N$23: now also RXI_5.1; no longer PAD6.1
- net PD2/RXI/D0: now also Q6.2, R17.1; no longer J1.2, J4.2
- net PD3/TXO/D1: now also Q5.2, R15.1; no longer J1.1, J4.1
- net RXA: now also J4.2, Q4.2, R13.1
- net RXB: now also J1.2, Q2.2, R9.1
- net TXA: now also J4.1, Q3.2, R11.1
- net TXB: now also J1.1, Q1.2, R7.1

Commit message: Fixed errors and relayed out, last attempt with MOSFET level shifter, need to try TXS shifter
Parts:
- moved RXA_5 20.3 mm to (25.5, 4.95)
- moved TXB_5 15.4 mm to (7.49, 4.95)
- moved TXO_5 15.4 mm to (23.0, 4.95)
- moved RXB_5 15.4 mm to (7.49, 2.54)
- moved RXI_5 15.4 mm to (23.0, 2.54)
- moved R2 11.9 mm to (9.02, 15.5)
- moved R1 11.8 mm to (20.7, 15.5)
- moved R12 6.31 mm to (8.38, 6.86), turned to 180 degrees
- moved R18 6.26 mm to (21.2, 6.86), turned to 0 degrees
- moved R8 4.34 mm to (8.38, 13.8)
- moved R14 4.27 mm to (21.2, 14.0), turned to 0 degrees
- moved R16 3.14 mm to (21.2, 10.4), turned to 0 degrees
- moved R10 3.07 mm to (8.38, 10.4)
- moved TXA_5 1.91 mm to (5.08, 4.95)
- moved R15 1.82 mm to (21.2, 12.2), turned to 0 degrees
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Connections:
- net N$3: no longer R2.2
- net N$5: now also R2.2
- net PB1/D15/SCK: now also J4.1; no longer J4.12
- net PB2/D16/MOSI: now also J4.2; no longer J4.11
- net PB3/D14/MISO: now also J4.3; no longer J4.10
- net PD0/SCL/D3: now also J4.9; no longer J4.4
- net PD1/SDA/D2: now also J4.10; no longer J4.3
- net PF0/A5: now also J4.4; no longer J4.9
- net RXA: now also J4.11; no longer J4.2
- net TXA: now also J4.12; no longer J4.1
Routing:
- net GND: track 0.00 -> 40.3 mm, vias 0 -> 2
- net 3V3: track 0.00 -> 22.7 mm
- net PD0/SCL/D3: track 0.00 -> 16.1 mm, vias 0 -> 1
- net N$3: track 0.00 -> 14.3 mm, vias 0 -> 2
- net RXB: track 0.00 -> 13.9 mm, vias 0 -> 2
- net TXB: track 0.00 -> 9.34 mm
- net N$17: track 0.00 -> 8.92 mm
- net TXA: track 0.00 -> 5.66 mm
- net N$5: track 0.00 -> 4.94 mm
- net N$19: track 0.00 -> 4.05 mm
- net N$22: track 0.00 -> 4.05 mm
- net N$20: track 0.00 -> 4.05 mm
- net N$23: track 0.00 -> 4.05 mm
- net N$21: track 0.00 -> 4.05 mm
- net N$18: track 0.00 -> 4.05 mm
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
Commit message: Added TXS based level translation
Parts:
- removed Q1, Q2, Q3, Q4, Q5, Q6: MOSFET-N-044020001, OPL:SOT23
- removed R10, R11, R12, R13, R14, R15, R16, R17, R18, R7, R8, R9: 10K, OPL:R0603
- removed RXA_5, RXB_5, RXI_5, TXA_5, TXB_5, TXO_5: WIREPAD1,6/0,8, wirepad:1,6/0,8
- added RXA, RXB, RXI, TXA, TXB, TXO: (no value), wirepad:1,6/0,8
- added U2: TXB0106PWR, Texas Instruments_By_element14_Batch_1:SOP65P640X120-16N
- 5V, GND: value WIREPAD1,6/0,8 -> (none)
- moved GND 12.9 mm to (19.8, 16.3), flipped to the top
- moved C1 9.96 mm to (21.3, 18.5), turned to 0 degrees
- moved R2 7.38 mm to (14.6, 20.3), turned to 180 degrees
- moved R1 6.87 mm to (14.6, 18.7), turned to 180 degrees
- moved C2 6.17 mm to (21.3, 20.2), turned to 0 degrees
- moved X1 5.34 mm to (18.0, 19.6), turned to 180 degrees
- moved S1 4.96 mm to (9.59, 19.6), turned to 270 degrees
- moved 5V 3.86 mm to (21.8, 16.3), flipped to the top
- moved D4 3.75 mm to (16.9, 3.81)
- moved R6 3.39 mm to (17.0, 2.35)
- moved D3 3.31 mm to (13.8, 3.81)
- moved D2 3.10 mm to (10.8, 3.81)
- moved D1 2.80 mm to (7.75, 3.81)
- moved R5 2.77 mm to (13.9, 2.35)
- moved R4 2.69 mm to (10.9, 2.22)
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Connections:
- removed net N$17: 5V.1, R10.2, R12.2, R14.2, R16.2, R18.2, R8.2
- new net N$4: 5V.1, U2.15
- net 3V3: now also U2.2, U2.8; no longer Q1.1, Q2.1, Q3.1, Q4.1, Q5.1, Q6.1, R11.2, R13.2, R15.2, R17.2, R7.2, R9.2
- net GND: now also U2.9
- net N$18: now also RXI.1, U2.16; no longer Q1.3, R8.1, TXB_5.1
- net N$19: now also TXO.1, U2.14; no longer Q2.3, R10.1, RXB_5.1
- net N$20: now also RXA.1, U2.13; no longer Q3.3, R12.1, TXA_5.1
- net N$21: now also TXA.1, U2.12; no longer Q4.3, R14.1, RXA_5.1
- net N$22: now also RXB.1, U2.11; no longer Q5.3, R16.1, TXO_5.1
- net N$23: now also TXB.1, U2.10; no longer Q6.3, R18.1, RXI_5.1
- net PB1/D15/SCK: no longer J1.12, J4.1
- net PB2/D16/MOSI: no longer J1.11, J4.2
- net PB3/D14/MISO: no longer J1.10, J4.3
- net PD0/SCL/D3: no longer J1.4, J4.9
- net PD1/SDA/D2: no longer J1.3, J4.10
- net PD2/RXI/D0: now also U2.1; no longer Q6.2, R17.1
- net PD3/TXO/D1: now also U2.3; no longer Q5.2, R15.1
- net PF0/A5: no longer J1.9, J4.4
- net RXA: now also U2.4; no longer Q4.2, R13.1
- net RXB: now also U2.6; no longer Q2.2, R9.1
- net TXA: now also U2.5; no longer Q3.2, R11.1
- net TXB: now also U2.7; no longer Q1.2, R7.1
Routing:
- net TXB: track 9.34 -> 66.5 mm, vias 0 -> 3
- net 3V3: track 22.7 -> 76.3 mm, vias 0 -> 7
- net TXA: track 5.66 -> 57.5 mm, vias 0 -> 4
- net GND: track 40.3 -> 88.8 mm, vias 2 -> 6
- net RXB: track 13.9 -> 49.7 mm, vias 2 -> 4
- net PD2/RXI/D0: track 1.65 -> 27.8 mm, vias 0 -> 3
- net RXA: track 1.65 -> 26.9 mm, vias 0 -> 3
- net PD3/TXO/D1: track 1.65 -> 25.8 mm, vias 0 -> 1
- net PD1/SDA/D2: track 0.00 -> 21.2 mm, vias 0 -> 4
- net PB1/D15/SCK: track 0.00 -> 18.1 mm
- net PB2/D16/MOSI: track 0.00 -> 18.0 mm
- net PB3/D14/MISO: track 0.00 -> 17.9 mm
- net PF0/A5: track 0.00 -> 17.6 mm, vias 0 -> 2
- net N$1: track 2.26 -> 16.5 mm, vias 0 -> 3
- net N$2: track 2.21 -> 14.9 mm, vias 0 -> 3
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Other:
- board text added: "by Tisham Dhar"
- board text removed: "by Seeed Studio"

Commit message: Changed to 5x3 crystal
Parts:
- removed X1: CTS_32X25_SMD, crystal-cts:CTS_32X25
- added Y1: (no value), SparkFun-FreqCtrl:CRYSTAL-SMD-5X3
- moved C1 1.91 mm to (23.2, 18.7)
- moved C2 1.91 mm to (23.2, 20.3)
Connections:
- net GND: no longer X1.2, X1.4
- net N$1: now also Y1.1; no longer X1.1
- net N$2: now also Y1.3; no longer X1.3
Routing:
- net GND: track 88.8 -> 82.9 mm, vias 6 -> 7
- net N$1: track 16.5 -> 14.5 mm, vias 3 -> 4
- net N$2: track 14.9 -> 14.7 mm, vias 3 -> 4

Commit message: Changed caps to match crystal load
Parts:
- C1: value 22pF -> 15pF
- C2: value 33pF -> 22pF
Routing:
- net GND: track 82.9 -> 83.8 mm
Changed lines of the file:
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@@
 <attribute name="VALUE" x="10.553" y="22.654" size="0.889" layer="28" ratio="11" rot="MR180"/>
 </element>
-<element name="C1" library="OPL" package="C0603" value="22pF" x="23.241" y="18.669" smashed="yes">
+<element name="C1" library="OPL" package="C0603" value="15pF" x="23.241" y="18.669" smashed="yes">
 <attribute name="NAME" x="25.781" y="18.669" size="0.508" layer="25" ratio="11" rot="R180"/>
-<attribute name="VALUE" x="24.511" y="18.9865" size="0.635" layer="27" ratio="10" rot="R180"/>
-</element>
-<element name="C2" library="OPL" package="C0603" value="33pF" x="23.241" y="20.32" smashed="yes">
+<attribute name="VALUE" x="23.0505" y="19.431" size="0.381" layer="27" ratio="10" rot="R270"/>
+</element>
+<element name="C2" library="OPL" package="C0603" value="22pF" x="23.241" y="20.32" smashed="yes">
 <attribute name="NAME" x="24.765" y="20.701" size="0.508" layer="25" ratio="11"/>
-<attribute name="VALUE" x="22.225" y="20.1295" size="0.635" layer="27" ratio="10"/>
+<attribute name="VALUE" x="23.4315" y="19.685" size="0.381" layer="27" ratio="10" rot="R90"/>
 </element>
 <element name="S1" library="switch-copal" package="CHS-02A" value="CHS-02A" x="9.5885" y="19.558" smashed="yes" rot="R270">
@@
 <wire x1="16.51" y1="16.256" x2="14.859" y2="17.907" width="0.3048" layer="1"/>
 <wire x1="19.812" y1="16.256" x2="16.51" y2="16.256" width="0.3048" layer="1"/>
-<wire x1="22.733" y1="17.272" x2="23.622" y2="17.272" width="0.3048" layer="1"/>
 <wire x1="22.479" y1="17.272" x2="22.733" y2="17.272" width="0.3048" layer="16"/>
 <wire x1="22.352" y1="17.399" x2="22.479" y2="17.272" width="0.3048" layer="16"/>
@@
 <wire x1="19.812" y1="16.256" x2="20.955" y2="17.399" width="0.3048" layer="16"/>
 <via x="22.733" y="17.272" extent="1-16" drill="0.3048"/>
-<wire x1="23.622" y1="17.272" x2="23.876" y2="17.526" width="0.3048" layer="1"/>
 <wire x1="22.225" y1="17.526" x2="22.225" y2="17.399" width="0.3048" layer="1"/>
 <wire x1="22.352" y1="17.653" x2="22.225" y2="17.526" width="0.3048" layer="1"/>
@@
 <wire x1="22.479" y1="20.32" x2="22.352" y2="20.32" width="0.3048" layer="1"/>
 <wire x1="22.352" y1="18.796" x2="22.479" y2="18.669" width="0.3048" layer="1"/>
+<wire x1="22.86" y1="17.145" x2="24.765" y2="17.145" width="0.3048" layer="1"/>
+<wire x1="22.733" y1="17.272" x2="22.86" y2="17.145" width="0.3048" layer="1"/>
 </signal>
 <signal name="PB1/D15/SCK">

Commit message: Added mini usb and mosfet based level shifter
Parts:
- removed RXA, RXB, RXI, TXA, TXB, TXO: (no value), wirepad:1,6/0,8
- removed Y1: (no value), SparkFun-FreqCtrl:CRYSTAL-SMD-5X3
- added R7: 10K, Discrete:1206-8-3.3X2.4
- added RXB_5, TXB_5: (no value), wirepad:1,6/0,8
- added X1: CTS_32X25_SMD, cts_crystal:CTS_32X25
- J1: value 12p 0.5mm bottom contact -> MINI-USB-5P-3400020P1; device template:12P-0.5 -> OPL Eagle Library:MINI-B-SMD
- U2: value TXB0106PWR -> BSS138PS; device Texas Instruments_By_element14_Batch_1:SOP65P640X120-16N -> NXP_By_element14_Batch_1:SOT65P210X110-6N
- moved C1 17.0 mm to (11.7, 6.22), turned to 270 degrees
- moved C2 15.2 mm to (17.1, 6.35), turned to 90 degrees
- moved 5V 13.8 mm to (23.5, 2.54)
- moved U2 10.2 mm to (17.7, 18.8), flipped to the top, turned to 90 degrees
- moved R4 6.73 mm to (17.6, 2.35)
- moved D2 6.73 mm to (17.5, 3.81)
- moved D3 5.72 mm to (8.13, 3.94)
- moved R5 5.72 mm to (8.19, 2.48)
- moved GND 4.21 mm to (23.5, 18.3)
- moved D4 3.81 mm to (20.7, 3.81)
- moved D1 3.69 mm to (11.4, 3.94)
- moved R6 3.68 mm to (20.6, 2.35)
- moved R3 3.57 mm to (11.4, 2.48)
- moved J1 2.41 mm to (14.7, 17.9)
- moved J4 2.16 mm to (14.6, 3.56)
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Connections:
- removed net N$18: RXI.1, U2.16
- removed net N$19: TXO.1, U2.14
- removed net N$20: RXA.1, U2.13
- removed net N$21: TXA.1, U2.12
- removed net N$22: RXB.1, U2.11
- removed net N$23: TXB.1, U2.10
- removed net N$4: 5V.1, U2.15
- new net 5V: 5V.1, J1.1, R7.1, R7.2
- new net GPIO0: J1.2, U1.18
- new net GPIO1: J1.4, U1.19
- new net RXB_5: R7.8, RXB_5.1, U2.6
- new net TXB_5: J1.3, R7.7, TXB_5.1, U2.3
- net 3V3: now also R7.5, R7.6, U2.5; no longer J1.5, J1.8, U2.8
- net GND: now also J1.5, J1.P$1, J1.P$2, J1.P$3, J1.P$4, X1.2, X1.4; no longer J1.6, J1.7, J1.P1, J1.P2, U2.9
- net N$1: now also X1.1; no longer Y1.1
- net N$2: now also X1.3; no longer Y1.3
- net PD2/RXI/D0: no longer U2.1
- net PD3/TXO/D1: no longer U2.3
- net RXA: no longer U2.4
- net RXB: now also R7.3, U2.1; no longer J1.2, U2.6
- net TXA: no longer U2.5
- net TXB: now also R7.4, U2.4; no longer J1.1, U2.7
Routing:
- net N$5: track 14.1 -> 56.7 mm, vias 0 -> 8
- net 5V: track 0.00 -> 40.3 mm, vias 0 -> 4
- net TXB_5: track 0.00 -> 39.4 mm, vias 0 -> 1
- net TXA: track 57.5 -> 21.0 mm
- net N$3: track 6.22 -> 34.2 mm, vias 0 -> 2
- net TXB: track 66.5 -> 38.8 mm
- net RXB: track 49.7 -> 33.4 mm, vias 4 -> 2
- net GPIO0: track 0.00 -> 16.1 mm, vias 0 -> 1
- net RXB_5: track 0.00 -> 14.9 mm, vias 0 -> 4
- net N$21: track 14.4 -> 0.00 mm
- net GND: track 83.8 -> 72.3 mm, vias 7 -> 17
- net PD2/RXI/D0: track 27.8 -> 16.8 mm, vias 3 -> 0
- net N$2: track 14.7 -> 4.78 mm, vias 4 -> 0
- net RXA: track 26.9 -> 36.5 mm, vias 3 -> 2
- net N$19: track 9.30 -> 0.00 mm, vias 1 -> 0
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Other:
- board text added: "v2.0 26/02/2015"
- board text removed: "v1.0 14/09/2014"
