File: Xadow MultiSerial.brd (EAGLE design)
At the start: 25.4 x 20.3 mm, 25 parts, among them J1 MINI-USB-5P-3400020P1, J2 12p 0.5mm bottom contact, J3 12p 0.5mm bottom contact, J4 12p 0.5mm bottom contact, U1 SC16IS752, U2 BSS138PS, X1 CTS_32X25_SMD

Commit message: Converted board to SPI
Parts:
- removed R1: 10k, OPL:R0603
- removed R2: 10K, OPL:R0603
- removed S1: CHS-02A, switch-copal:CHS-02A
Connections:
- removed net N$3: R1.2, S1.3, U1.11
- removed net N$5: R2.2, S1.4, U1.10
- net 3V3: no longer S1.1, S1.2, U1.9
- net GND: now also U1.14, U1.9; no longer R1.1, R2.1
- net PB1/D15/SCK: now also U1.13
- net PB2/D16/MOSI: now also U1.11
- net PB3/D14/MISO: now also U1.12
- net PD0/SCL/D3: no longer U1.13
- net PD1/SDA/D2: no longer U1.14
- net PF0/A5: now also U1.10
Routing:
- net N$5: track 56.7 -> 0.00 mm, vias 8 -> 0
- net PB3/D14/MISO: track 16.0 -> 52.6 mm, vias 0 -> 2
- net N$3: track 34.2 -> 0.00 mm, vias 2 -> 0
- net PB2/D16/MOSI: track 16.1 -> 50.3 mm, vias 0 -> 2
- net PF0/A5: track 15.9 -> 33.5 mm
- net PB1/D15/SCK: track 16.3 -> 33.5 mm
- net PD0/SCL/D3: track 24.9 -> 16.5 mm, vias 2 -> 0
- net RXA: track 36.5 -> 28.6 mm, vias 2 -> 1
- net 3V3: track 80.2 -> 76.4 mm, vias 11 -> 9
- net GND: track 72.3 -> 75.9 mm, vias 17 -> 18
- net PD1/SDA/D2: track 19.9 -> 16.7 mm, vias 2 -> 0
- net GPIO1: track 4.14 -> 3.42 mm

Commit message: Added a 3V3 LDO to grab power
Parts:
- added C3, C4: 10uF, adafruit:C0805K
- added IC2: LP298XS, adafruit:SOT23-5L
Connections:
- removed net 3V3: D1.+, D2.+, D3.+, D4.+, J2.5, J2.8, J3.5, J3.8, J4.5, J4.8, R7.5, R7.6, U1.5, U1.8, U2.2, U2.5
- removed net 5V: 5V.1, J1.1, R7.1, R7.2
- new net +3V3: C3.1, C4.1, D1.+, D2.+, D3.+, D4.+, IC2.5, J2.5, J2.8, J3.5, J3.8, J4.5, J4.8, R7.5, R7.6, U1.5, U1.8, U2.2, U2.5
- new net +5V: 5V.1, IC2.1, IC2.3, J1.1, R7.1, R7.2
- net GND: now also C3.2, C4.2, IC2.2
Routing:
- net +3V3: track 0.00 -> 92.6 mm, vias 0 -> 11
- net 3V3: track 76.4 -> 0.00 mm, vias 9 -> 0
- net +5V: track 0.00 -> 55.4 mm, vias 0 -> 6
- net 5V: track 40.3 -> 0.00 mm, vias 4 -> 0
- net GND: track 75.9 -> 72.6 mm, vias 18 -> 17
Changed lines of the file:
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@@
 <layer number="23" name="tOrigins" color="15" fill="1" visible="yes" active="yes"/>
 <layer number="24" name="bOrigins" color="3" fill="1" visible="yes" active="yes"/>
-<layer number="25" name="tNames" color="7" fill="1" visible="yes" active="yes"/>
-<layer number="26" name="bNames" color="3" fill="1" visible="yes" active="yes"/>
+<layer number="25" name="tNames" color="7" fill="1" visible="no" active="yes"/>
+<layer number="26" name="bNames" color="3" fill="1" visible="no" active="yes"/>
 <layer number="27" name="tValues" color="7" fill="1" visible="no" active="yes"/>
 <layer number="28" name="bValues" color="7" fill="1" visible="no" active="yes"/>
@@
 </element>
 <element name="R7" library="Discrete" package="1206-8-3.3X2.4" value="10K" x="20.701" y="19.05" rot="R180"/>
+<element name="C3" library="adafruit" package="C0805K" value="10uF" x="13.335" y="19.05" rot="R90"/>
+<element name="C4" library="adafruit" package="C0805K" value="10uF" x="7.62" y="19.05" rot="R90"/>
+<element name="IC2" library="adafruit" package="SOT23-5L" value="LP298XS" x="10.541" y="19.05" rot="R90"/>
 </elements>
 <signals>
-<signal name="3V3" class="2">
+<signal name="+3V3" class="2">
 <contactref element="J2" pad="5"/>
 <contactref element="J2" pad="8"/>
@@
 <wire x1="13.589" y1="7.366" x2="13.4874" y2="7.2644" width="0.3048" layer="16"/>
 <wire x1="15.367" y1="5.969" x2="15.355" y2="5.906" width="0.3048" layer="16"/>
+<contactref element="C3" pad="1"/>
+<contactref element="C4" pad="1"/>
+<contactref element="IC2" pad="5"/>
+<wire x1="8.382" y1="18.1102" x2="9.2202" y2="18.1102" width="0.3048" layer="1"/>
+<wire x1="8.3312" y1="18.0594" x2="8.382" y2="18.1102" width="0.3048" layer="1"/>
+<wire x1="7.62" y1="18.0594" x2="8.3312" y2="18.0594" width="0.3048" layer="1"/>
+<wire x1="9.2202" y1="18.1102" x2="9.241" y2="18.1" width="0.3048" layer="1"/>
+<wire x1="7.62" y1="18.0594" x2="7.62" y2="18.05" width="0.3048" layer="1"/>
+<wire x1="12.8016" y1="18.0594" x2="13.335" y2="18.0594" width="0.3048" layer="1"/>
+<wire x1="12.8016" y1="17.4752" x2="12.8016" y2="18.0594" width="0.3048" layer="1"/>
+<wire x1="12.7762" y1="17.4498" x2="12.8016" y2="17.4752" width="0.3048" layer="1"/>
+<wire x1="10.5918" y1="17.4498" x2="12.7762" y2="17.4498" width="0.3048" layer="1"/>
+<wire x1="9.9314" y1="18.1102" x2="10.5918" y2="17.4498" width="0.3048" layer="1"/>
+<wire x1="9.398" y1="18.1102" x2="9.9314" y2="18.1102" width="0.3048" layer="1"/>
+<wire x1="13.335" y1="18.0594" x2="13.335" y2="18.05" width="0.3048" layer="1"/>
+<wire x1="9.398" y1="18.1102" x2="9.241" y2="18.1" width="0.3048" layer="1"/>
+<wire x1="7.1628" y1="18.0594" x2="7.493" y2="18.0594" width="0.3048" layer="1"/>
+<wire x1="7.1628" y1="17.3228" x2="7.1628" y2="18.0594" width="0.3048" layer="1"/>
+<wire x1="7.3406" y1="17.145" x2="7.1628" y2="17.3228" width="0.3048" layer="1"/>
+<wire x1="7.3406" y1="15.9258" x2="7.3406" y2="17.145" width="0.3048" layer="1"/>
+<wire x1="4.5974" y1="13.1826" x2="7.3406" y2="15.9258" width="0.3048" layer="1"/>
+<wire x1="4.5974" y1="12.9794" x2="4.5974" y2="13.1826" width="0.3048" layer="1"/>
+<wire x1="5.588" y1="11.9888" x2="4.5974" y2="12.9794" width="0.3048" layer="16"/>
+<wire x1="6.223" y1="11.9888" x2="5.588" y2="11.9888" width="0.3048" layer="1"/>
+<wire x1="6.2992" y1="12.065" x2="6.223" y2="11.9888" width="0.3048" layer="1"/>
+<wire x1="6.8326" y1="12.065" x2="6.2992" y2="12.065" width="0.3048" layer="1"/>
+<wire x1="7.493" y1="18.0594" x2="7.62" y2="18.05" width="0.3048" layer="1"/>
+<wire x1="6.8326" y1="12.065" x2="6.9855" y2="12.053" width="0.3048" layer="1"/>
+<via x="4.5974" y="12.9794" extent="1-16" drill="0.3048"/>
+<via x="5.588" y="11.9888" extent="1-16" drill="0.3048"/>
 </signal>
 <signal name="GND">
@@
 <wire x1="8.8265" y1="15.4305" x2="7.62" y2="16.637" width="0.3048" layer="16"/>
 <wire x1="10.16" y1="14.097" x2="10.232" y2="14.01" width="0.3048" layer="16"/>
-<wire x1="6.477" y1="16.637" x2="6.223" y2="16.637" width="0.3048" layer="16"/>
 <wire x1="6.731" y1="16.891" x2="6.477" y2="16.637" width="0.3048" layer="16"/>
 <wire x1="6.223" y1="16.383" x2="6.731" y2="16.891" width="0.3048" layer="1"/>
@@
 <wire x1="4.7625" y1="6.223" x2="5.207" y2="6.223" width="0.3048" layer="1"/>
 <via x="6.604" y="4.826" extent="1-16" drill="0.3048"/>
-<wire x1="6.858" y1="18.669" x2="6.858" y2="18.719796875" width="0.1524" layer="16"/>
-<wire x1="5.334" y1="17.526" x2="5.2901125" y2="17.569890625" width="0.1524" layer="16"/>
 <wire x1="16.9418" y1="5.715" x2="17.145" y2="5.588" width="0.1524" layer="1"/>
 <wire x1="16.9418" y1="5.715" x2="17.049728125" y2="5.68325" width="0.1524" layer="1"/>
@@
 <wire x1="9.779" y1="16.383" x2="9.906" y2="16.383" width="0.3048" layer="1"/>
 <wire x1="8.8265" y1="15.4305" x2="9.779" y2="16.383" width="0.3048" layer="16"/>
-<wire x1="9.906" y1="17.653" x2="9.906" y2="16.383" width="0.3048" layer="1"/>
-<wire x1="8.763" y1="18.796" x2="9.906" y2="17.653" width="0.3048" layer="1"/>
 <via x="9.779" y="16.383" extent="1-16" drill="0.3048"/>
-<via x="8.763" y="18.796" extent="1-16" drill="0.3048"/>
 <via x="14.605" y="20.701" extent="1-16" drill="0.3048"/>
-<via x="13.208" y="17.399" extent="1-16" drill="0.3048"/>
+<via x="13.589" y="17.018" extent="1-16" drill="0.3048"/>
 <wire x1="10.0838" y1="5.6896" x2="10.16" y2="5.715" width="0.1524" layer="1"/>
 <wire x1="9.4234" y1="3.6322" x2="9.525" y2="3.683" width="0.1524" layer="16"/>
@@
 <wire x1="15.748" y1="8.763" x2="15.7705" y2="8.784" width="0.3048" layer="1"/>
 <via x="15.494" y="7.62" extent="1-16" drill="0.3048"/>
+<contactref element="C3" pad="2"/>
+<contactref element="C4" pad="2"/>
+<contactref element="IC2" pad="2"/>
 </signal>
 <signal name="PB1/D15/SCK">
@@
 <wire x1="19.9898" y1="2.2352" x2="19.8755" y2="2.3495" width="0.1524" layer="1"/>
 </signal>
-<signal name="5V">
+<signal name="+5V">
 <contactref element="R7" pad="1"/>
 <contactref element="R7" pad="2"/>
@@
 <via x="23.9522" y="13.97" extent="1-16" drill="0.3048"/>
 <via x="22.3012" y="15.9258" extent="1-16" drill="0.3048"/>
+<contactref element="IC2" pad="1"/>
+<contactref element="IC2" pad="3"/>
+<wire x1="11.2014" y1="18.1102" x2="11.8364" y2="18.1102" width="0.1524" layer="1"/>
+<wire x1="10.9474" y1="18.3642" x2="11.2014" y2="18.1102" width="0.1524" layer="1"/>
+<wire x1="10.9474" y1="19.7866" x2="10.9474" y2="18.3642" width="0.1524" layer="1"/>
+<wire x1="11.1506" y1="19.9898" x2="10.9474" y2="19.7866" width="0.1524" layer="1"/>
+<wire x1="11.8364" y1="19.9898" x2="11.1506" y2="19.9898" width="0.1524" layer="1"/>
+<wire x1="11.8364" y1="18.1102" x2="11.841" y2="18.1" width="0.1524" layer="1"/>
+<wire x1="11.8364" y1="19.9898" x2="11.841" y2="20" width="0.1524" layer="1"/>
+<wire x1="12.2936" y1="19.9898" x2="11.9126" y2="19.9898" width="0.1524" layer="1"/>
+<wire x1="12.2936" y1="20.6248" x2="12.2936" y2="19.9898" width="0.1524" layer="1"/>
+<wire x1="12.1666" y1="20.7518" x2="12.2936" y2="20.6248" width="0.1524" layer="1"/>
+<wire x1="13.8684" y1="19.05" x2="12.1666" y2="20.7518" width="0.1524" layer="16"/>
+<wire x1="14.2494" y1="19.05" x2="13.8684" y2="19.05" width="0.1524" layer="16"/>
+<wire x1="14.5288" y1="19.05" x2="14.2494" y2="19.05" width="0.1524" layer="1"/>
+<wire x1="16.4592" y1="20.9804" x2="14.5288" y2="19.05" width="0.1524" layer="1"/>
+<wire x1="20.6248" y1="20.9804" x2="16.4592" y2="20.9804" width="0.1524" layer="1"/>
+<wire x1="20.955" y1="20.6502" x2="20.6248" y2="20.9804" width="0.1524" layer="1"/>
+<wire x1="11.9126" y1="19.9898" x2="11.841" y2="20" width="0.1524" layer="1"/>
+<via x="12.1666" y="20.7518" extent="1-16" drill="0.3048"/>
+<via x="14.2494" y="19.05" extent="1-16" drill="0.3048"/>
 </signal>
 <signal name="RXB_5">
